File: hardware/firefly2.sch (KiCad schematic (older format))
At the start: 20 parts, among them J1 10118194-0001LF, P2 CONN_01X03, P3 CONN_01X04, P4 CONN_01X05, P5 CONN_01X01, U1 SAM_D11C, U2 RFM69CW, U3 MIC5504

Commit message: Place v2.1 parts (no routing yet)
Change-Id: I3c64d8efe2df87153508bcfdb10d42841a7add0c
Parts:
- removed J1: 10118194-0001LF, 10118194-0001LF:FRAMATOME_10118194-0001LF, symbol 10118194-0001LF
- removed P2: CONN_01X03, SparkFun-Connectors:1X03, symbol CONN_01X03
- removed R1: 220, SparkFun-Resistors:0603, symbol R
- removed U1: SAM_D11C, SMD_Packages:SOIC-14_N, symbol SAM_D11C
- added U1: SAMD21E18, SparkFun-DigitalIC:TQFP32-08, symbol SAMD21E18
- gave numbers to parts that had none: 2
Connections:
- wire segments 22 -> 27
- no-connect marks 7 -> 22
Other:
- note added: "Replace the CPU\nSwitch 3v3 to 5v on programming header\nDitch off board led header\nDitch aux pins\nAdd debugging via for serial LEDs (Processor out goes to led and add a via to the line in case we need a logic probe to analyze it and it can be super tiny)\nSilkscreen might be wrong (radio iconography is backward maybe)\nRemove resistor for 1wire LEDs\n"
- note removed: "Off board LED"

Commit message: Fix radio silkscreen orientation for v2.1
Change-Id: I934a96829cceb58ae09e96efa49570f37a8bb193
Parts:
- J2: footprint 10118194-0001LF:FRAMATOME_10118194-0001LF -> Connector_USB:USB_Micro-B_Wuerth-614105150721_Vertical
- U2: footprint homebrew:RFM69CW-XXXS2 -> homebrew:RFM69CW
Changed lines of the file:
@@
 LIBS:contrib
 LIBS:valves
-LIBS:homebrew
-LIBS:GeekAmmo
-LIBS:LilyPad-Wearables
-LIBS:SparkFun-Aesthetics
-LIBS:SparkFun-AnalogIC
-LIBS:SparkFun-Boards
-LIBS:SparkFun-Capacitors
-LIBS:SparkFun-Connectors
-LIBS:SparkFun-DigitalIC
-LIBS:SparkFun-DiscreteSemi
-LIBS:SparkFun-Displays
-LIBS:SparkFun-Electromechanical
-LIBS:SparkFun-FreqCtrl
-LIBS:SparkFun-LED
-LIBS:SparkFun-Passives
-LIBS:SparkFun-PowerIC
-LIBS:SparkFun-Resistors
-LIBS:SparkFun-Retired
-LIBS:SparkFun-RF
-LIBS:SparkFun-Sensors
-LIBS:Teensy_3_and_LC_Series_Boards_v1.1
-LIBS:User-Submitted
-LIBS:adafruit
-LIBS:10118194-0001LF
 LIBS:firefly2-cache
 EELAYER 25 0
@@
 F 0 "U2" H 4500 2250 50  0000 L BNN
 F 1 "RFM69CW" H 4500 1075 50  0000 L BNN
-F 2 "homebrew:RFM69CW-XXXS2" H 4930 1850 20  0001 C CNN
+F 2 "homebrew:RFM69CW" H 4930 1850 20  0001 C CNN
 F 3 "" H 4900 1700 60  0000 C CNN
 	1    4900 1700
@@
 F 0 "J2" H 1209 6721 50  0000 L BNN
 F 1 "614105150721" H 1199 6199 50  0000 L BNN
-F 2 "10118194-0001LF:FRAMATOME_10118194-0001LF" H 1500 6500 50  0001 L BNN
+F 2 "Connector_USB:USB_Micro-B_Wuerth-614105150721_Vertical" H 1500 6500 50  0001 L BNN
 F 3 "Amphenol" H 1500 6500 50  0001 L BNN
 F 4 "0.25 USD" H 1500 6500 50  0001 L BNN "Field4"
