File: hardware/controller/controller.sch (KiCad schematic (older format))
At the start: 60 parts

Commit message: First pass of controller schematic complete
Change-Id: Ie86e1f4b393c798507bb2ab72719fa5d4e7f3f36
Parts:
- added C1, C3, C5, C6: 0.1uF, Capacitor_SMD:C_0402_1005Metric_Pad0.74x0.62mm_HandSolder, symbol Device:C
- added C10, C2, C4, C8: 4.7uF, Capacitor_SMD:C_0603_1608Metric, symbol Device:C
- added C19: 1pF, Capacitor_SMD:C_0402_1005Metric_Pad0.74x0.62mm_HandSolder, symbol Device:C
- added D1, D2, D26, D3, D30, D31, D4, D46: D_TVS, Diode_SMD:D_SOD-323, symbol Device:D_TVS
- added J1: Conn_01x05, Connector_PinHeader_2.54mm:PinHeader_1x05_P2.54mm_Vertical, symbol Connector_Generic:Conn_01x05
- added J3: Conn_01x04, Connector_PinHeader_2.54mm:PinHeader_1x04_P2.54mm_Vertical, symbol Connector_Generic:Conn_01x04
- added J4: USB_B_Micro, homebrew:FRAMATOME_10118194-0001LF_fixed_bridges, symbol Connector:USB_B_Micro
- added JP1: SolderJumper_2_Open, Jumper:SolderJumper-2_P1.3mm_Open_RoundedPad1.0x1.5mm, symbol Jumper:SolderJumper_2_Open
- added L1: 10nH, Inductor_SMD:L_0402_1005Metric, symbol Device:L
- added R1, R11, R25, R7: 33R, Resistor_SMD:R_0603_1608Metric, symbol Device:R
- added R10, R13, R6: 100R, Resistor_SMD:R_0603_1608Metric, symbol Device:R
- added R12, R14, R15, R16, R17, R18, R22, R23, R24: 0R, Resistor_SMD:R_0603_1608Metric, symbol Device:R
- added R19, R26, R3: 47k, Resistor_SMD:R_0603_1608Metric, symbol Device:R
- added R2: 470k, Resistor_SMD:R_0603_1608Metric, symbol Device:R
- added R20, R27, R4: 24k, Resistor_SMD:R_0603_1608Metric, symbol Device:R
- added R21, R28, R5: 68k, Resistor_SMD:R_0603_1608Metric, symbol Device:R
- added R8: 240k, Resistor_SMD:R_0603_1608Metric, symbol Device:R
- added R9: 680k, Resistor_SMD:R_0603_1608Metric, symbol Device:R
- added S1: OS103011MS8QP1, OS102011MS8QP1, symbol snapeda-OS103011MS8QP1:OS103011MS8QP1
- added SW1, SW2, SW3, SW4, SW5, SW6, SW7, SW8, SW9: ILS_TA180_50, homebrew:SW_CK_TA, symbol Homebrew:ILS_TA180_50
- added U1, U3, U4: WS2811, Package_SO:SOP-8_3.9x4.9mm_P1.27mm, symbol Homebrew:WS2811
- J2: renamed from J?; value Conn_01x02 -> Conn_01x03; footprint (none) -> Connector_PinHeader_2.54mm:PinHeader_1x03_P2.54mm_Horizontal; symbol Connector_Generic:Conn_01x02 -> Connector_Generic:Conn_01x03
- SW10: renamed from SW?; footprint (none) -> homebrew:ANR11R11P2HQE; MPN (none) -> ANR11R11P2HQE
- U7: renamed from U?; LCSC (none) -> C382139
- gave numbers to parts that had none: 57
Connections:
- net labels added: AUX0, AUX1, BLED_0, BLED_1, BLED_2, BLED_3, BLED_4, BLED_5, BLED_6, BLED_7, BLED_8, LED_OUT, SWCLK, SWDIO, SW_ACTION, SW_LEFT, SW_MODE, SW_RIGHT
- wire segments 138 -> 276
- no-connect marks 7 -> 37
Other:
- note added: "Action buttons"
- note added: "Left buttons"
- note added: "Right buttons"
- moved on the sheet: C11, C12, C13, C14, C15, C16, C17, C18, C7, C9, D10, D11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

Commit message: Rough layout - user interface
Change-Id: I897ce85222109fb351b7544bab62b02ff1907d44
Parts:
- added D47, D48, D49: WS2812B, LED_SMD:LED_WS2812B_PLCC4_5.0x5.0mm_P3.2mm, symbol LED:WS2812B
- added H1, H2, H3, H4: MountingHole, MountingHole:MountingHole_3.2mm_M3, symbol Mechanical:MountingHole
- S1: footprint OS102011MS8QP1 -> snapeda:OS102011MS8QP1
- U6: footprint RFM69CW-XXXS2 -> homebrew:RFM69CW-minimalpads
Connections:
- net +BATT: now also D47.1 (VDD), D48.1 (VDD), D49.1 (VDD)
- net GND: now also D47.3 (VSS), D48.3 (VSS), D49.3 (VSS)
- net at D45.2 (DOUT): now also D47.4 (DIN)
- new net: D47.2 (DOUT), D48.4 (DIN)
- new net: D48.2 (DOUT), D49.4 (DIN)
Other:
- moved on the sheet: D12, D15, D18, D21, D24, D28, D33, D37, D41, D44, D6, D9

Commit message: Add controller antenna
Parts:
- S1: symbol snapeda-OS103011MS8QP1:OS103011MS8QP1 -> controller-rescue:OS103011MS8QP1-snapeda-OS103011MS8QP1
- SW1, SW2, SW3, SW4, SW5, SW6, SW7, SW8, SW9: symbol Homebrew:ILS_TA180_50 -> controller-rescue:ILS_TA180_50-Homebrew
- U1, U3, U4: symbol Homebrew:WS2811 -> controller-rescue:WS2811-Homebrew
- U2: symbol snapeda-STM32G031F8P6:STM32G031F8P6 -> controller-rescue:STM32G031F8P6-snapeda-STM32G031F8P6
- U6: symbol SparkFun-RF:RFM69CW-915MHZ -> controller-rescue:RFM69CW-915MHZ-SparkFun-RF
- U7: symbol snapeda-TP4056:TP4056 -> controller-rescue:TP4056-snapeda-TP4056
Changed lines of the file:
@@
 $EndDescr
 $Comp
-L snapeda-STM32G031F8P6:STM32G031F8P6 U2
+L controller-rescue:STM32G031F8P6-snapeda-STM32G031F8P6 U2
 U 1 1 624BA5CF
 P 2350 2050
@@
 Connection ~ 6350 15150
 $Comp
-L SparkFun-RF:RFM69CW-915MHZ U6
+L controller-rescue:RFM69CW-915MHZ-SparkFun-RF U6
 U 1 1 62516233
 P 13450 7350
@@
 Connection ~ 6350 14550
 $Comp
-L snapeda-TP4056:TP4056 U7
+L controller-rescue:TP4056-snapeda-TP4056 U7
 U 1 1 62620201
 P 14100 1600
@@
 	1100 2750 1150 2750
 $Comp
-L Homebrew:ILS_TA180_50 SW1
+L controller-rescue:ILS_TA180_50-Homebrew SW1
 U 1 1 6255A351
 P 2500 5350
@@
 $EndComp
 $Comp
-L Homebrew:WS2811 U1
+L controller-rescue:WS2811-Homebrew U1
 U 1 1 6257E8A0
 P 1900 12150
@@
 LED_OUT
 $Comp
-L Homebrew:WS2811 U3
+L controller-rescue:WS2811-Homebrew U3
 U 1 1 625ECF8B
 P 2450 13550
@@
 BLED_5
 $Comp
-L Homebrew:WS2811 U4
+L controller-rescue:WS2811-Homebrew U4
 U 1 1 626193EA
 P 3000 14950
@@
 	10100 3900 10100 3000
 $Comp
-L Homebrew:ILS_TA180_50 SW2
+L controller-rescue:ILS_TA180_50-Homebrew SW2
 U 1 1 62A31548
 P 2500 6350
@@
 NoConn ~ 2800 6550
 $Comp
-L Homebrew:ILS_TA180_50 SW3
+L controller-rescue:ILS_TA180_50-Homebrew SW3
 U 1 1 62A55D33
 P 2500 7350
@@
 Left buttons
 $Comp
-L Homebrew:ILS_TA180_50 SW4
+L controller-rescue:ILS_TA180_50-Homebrew SW4
 U 1 1 62E327B7
 P 4850 5400
@@
 NoConn ~ 5150 5600
 $Comp
-L Homebrew:ILS_TA180_50 SW5
+L controller-rescue:ILS_TA180_50-Homebrew SW5
 U 1 1 62E32F54
 P 4850 6400
@@
 NoConn ~ 5150 6600
 $Comp
-L Homebrew:ILS_TA180_50 SW6
+L controller-rescue:ILS_TA180_50-Homebrew SW6
 U 1 1 62E32F6D
 P 4850 7400
@@
 SW_ACTION
 $Comp
-L Homebrew:ILS_TA180_50 SW7
+L controller-rescue:ILS_TA180_50-Homebrew SW7
 U 1 1 62E58EFF
 P 7200 5400
@@
 NoConn ~ 7500 5600
 $Comp
-L Homebrew:ILS_TA180_50 SW8
+L controller-rescue:ILS_TA180_50-Homebrew SW8
 U 1 1 62E594BA
 P 7200 6400
@@
 NoConn ~ 7500 6600
 $Comp
-L Homebrew:ILS_TA180_50 SW9
+L controller-rescue:ILS_TA180_50-Homebrew SW9
 U 1 1 62E594D3
 P 7200 7400
@@
 Action buttons
 $Comp
-L snapeda-OS103011MS8QP1:OS103011MS8QP1 S1
+L controller-rescue:OS103011MS8QP1-snapeda-OS103011MS8QP1 S1
 U 1 1 62E839EF
 P 1100 9150

Commit message: Switch to STM32F103
Change-Id: I84217aec2ff83f4d57970417b635599fe3cc7776
Parts:
- removed U2: STM32G031F8P6, Package_SO:TSSOP-20_4.4x6.5mm_P0.65mm, symbol controller-rescue:STM32G031F8P6-snapeda-STM32G031F8P6
- added C20: 4.7uF, Capacitor_SMD:C_0603_1608Metric, symbol Device:C
- added C21, C22, C23, C24: 0.1uF, Capacitor_SMD:C_0402_1005Metric_Pad0.74x0.62mm_HandSolder, symbol Device:C
- added JP2: SolderJumper_2_Open, Jumper:SolderJumper-2_P1.3mm_Open_RoundedPad1.0x1.5mm, symbol Jumper:SolderJumper_2_Open
- added R34: 24k, Resistor_SMD:R_0603_1608Metric, symbol Device:R
- added U2: STM32F103C8Tx, Package_QFP:LQFP-48_7x7mm_P0.5mm, symbol MCU_ST_STM32F1:STM32F103C8Tx
Connections:
- net AUX0: now also U2.18 (PB0)
- net AUX1: now also U2.19 (PB1)
- net DIO0: now also U2.26 (PB13)
- net GND: now also C20.1, C20.2, C21.1, C21.2, C22.1, C22.2, C23.1, C23.2, C24.1, JP2.1 (A), R34.1, U2.23 (VSS), U2.24 (VDD), U2.35 (VSS), U2.36 (VDD), U2.47 (VSS), U2.48 (VDD), U2.8 (VSSA), U2.9 (VDDA)
- net LED_OUT: now also U2.28 (PB15)
- net MISO: now also U2.16 (PA6)
- net MOSI: now also U2.17 (PA7)
- net NSS: now also U2.14 (PA4)
- net SCK: now also U2.15 (PA5)
- net SWCLK: now also U2.37 (PA14)
- net SWDIO: now also U2.34 (PA13)
- net SW_ACTION: now also U2.12 (PA2)
- net SW_LEFT: now also U2.10 (PA0)
- net SW_RIGHT: now also U2.11 (PA1)
- net VBATT_DIV: now also U2.13 (PA3)
- net at C1.2, JP1.1 (A): now also U2.7 (NRST)
- net USB-: now reaches J4.2 (D-)
- net USB-: now also U2.32 (PA11)
- net USB+: now reaches J4.3 (D+)
- net USB+: now also U2.33 (PA12)
- new net BOOT0: C24.2, JP2.2 (B), R34.2, U2.44 (BOOT0)
- no-connect marks 37 -> 54
Other:
- moved on the sheet: C1, C10, C2, C4, C7, C8, C9, D1, D2, D3, D4, D46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

Commit message: Controller layout first pass complete
Parts:
- added C25: 0.1uF, Capacitor_SMD:C_0402_1005Metric_Pad0.74x0.62mm_HandSolder, symbol Device:C
- added D50, D51: D_TVS, Diode_SMD:D_SOD-323, symbol Device:D_TVS
- C10, C2, C4, C8: value 4.7uF -> 0.1uF; footprint Capacitor_SMD:C_0603_1608Metric -> Capacitor_SMD:C_0402_1005Metric_Pad0.74x0.62mm_HandSolder; LCSC C19666 -> C307331
- D35: value RED -> GREEN; LCSC C2286 -> (none); MPN (none) -> LTST-C190KGKT
- U7: footprint SOP127P600X175-9N -> snapeda:SOP127P600X175-9N
Connections:
- net BLED_3: now also R22.1; no longer R15.1
- net BLED_5: now also R15.1; no longer R22.1
- net BLED_6: now also R23.1; no longer R18.1
- net BLED_7: now also R18.1; no longer R23.1
- net GND: now also C10.1, C4.2, SW1.4, SW2.4, SW3.4, SW4.4, SW5.4, SW6.4, SW7.4, SW8.4, SW9.4, C25.2, D50.2 (A2), D51.2 (A2); no longer C10.2, C14.2, C15.1, C16.2, C20.2, C21.2, C22.1, C23.1, C4.1, C7.2, C9.1, D31.1 (A1), J1.4 (Pin_4), J3.1 (Pin_1), JP2.1 (A), R19.2, R2.2, R26.2, R3.2, SW1.2, SW2.2, SW3.2, SW4.2, SW5.2, SW6.2, SW7.2, SW8.2, SW9.2, U2.24 (VDD), U2.36 (VDD), U2.48 (VDD), U2.9 (VDDA), U5.3 (VOUT), U6.2 (3.3V)
- net LED_OUT: now also D5.4 (DIN); no longer R1.2
- net SW_ACTION: now also C8.1; no longer C10.1
- net SW_MODE: now also C10.2; no longer C4.2
- net SW_RIGHT: now also C4.1; no longer C8.1
- net USB+: now also D51.1 (A1)
- net USB-: now also D50.1 (A1)
- net at R25.1: now also D47.4 (DIN); no longer D5.4 (DIN)
- net at D45.2 (DOUT): now also R7.2; no longer D47.4 (DIN)
- net at U1.5 (DO): no longer R7.2
- net at U3.5 (DO): now also R25.2; no longer R11.2
- net at U4.5 (DO): now also R1.2; no longer R25.2
- net at D49.2 (DOUT): now also R11.2
- new net VCC: C14.2, C15.1, C16.2, C20.2, C21.2, C22.1, C23.1, C25.1, C7.2, C9.1, D31.1 (A1), J1.4 (Pin_4), J3.1 (Pin_1), JP2.1 (A), R19.2, R2.2, R26.2, R3.2, U2.24 (VDD), U2.36 (VDD), U2.48 (VDD), U2.9 (VDDA), U5.3 (VOUT), U6.2 (3.3V)
Other:
- moved on the sheet: C11, C12, C14, C20, C3, C5, C6, D10, D11, D12, D13, D14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

Commit message: Controller final hardware v1.0
Change-Id: I90847cb8d53445091bda4f38bed38da399b968f0
Parts:
- added J5: Conn_01x03, Connector_PinHeader_2.54mm:PinHeader_1x03_P2.54mm_Horizontal, symbol Connector_Generic:Conn_01x03
- added R35: 33R, Resistor_SMD:R_0603_1608Metric, symbol Device:R
Connections:
- net +BATT: now also J5.1 (Pin_1)
- net GND: now also J5.3 (Pin_3)
- net at U1.5 (DO): now also R35.2
- new net: J5.2 (Pin_2), R35.1
- no-connect marks 54 -> 53
Changed lines of the file:
@@
 NoConn ~ 2150 8000
-Wire Notes Line
-	800  15700 800  10900
 Wire Notes Line
 	12050 2600 12050 550
@@
 Wire Wire Line
 	14400 13000 14550 13000
-NoConn ~ 15200 14700
 NoConn ~ 2750 7700
 Wire Wire Line
@@
 	0    1    1    0
 $EndComp
+$Comp
+L Connector_Generic:Conn_01x03 J5
+U 1 1 625CB373
+P 15500 15600
+F 0 "J5" H 15580 15642 50  0000 L CNN
+F 1 "Conn_01x03" H 15580 15551 50  0000 L CNN
+F 2 "Connector_PinHeader_2.54mm:PinHeader_1x03_P2.54mm_Horizontal" H 15500 15600 50  0001 C CNN
+F 3 "~" H 15500 15600 50  0001 C CNN
+	1    15500 15600
+	1    0    0    -1
+$EndComp
+$Comp
+L power:+BATT #PWR055
+U 1 1 625CBA25
+P 15250 15450
+F 0 "#PWR055" H 15250 15300 50  0001 C CNN
+F 1 "+BATT" H 15265 15623 50  0000 C CNN
+F 2 "" H 15250 15450 50  0001 C CNN
+F 3 "" H 15250 15450 50  0001 C CNN
+	1    15250 15450
+	1    0    0    -1
+$EndComp
+Wire Wire Line
+	15250 15450 15250 15500
+Wire Wire Line
+	15250 15500 15300 15500
+$Comp
+L power:GND #PWR076
+U 1 1 625EF1D6
+P 15250 15750
+F 0 "#PWR076" H 15250 15500 50  0001 C CNN
+F 1 "GND" H 15255 15577 50  0000 C CNN
+F 2 "" H 15250 15750 50  0001 C CNN
+F 3 "" H 15250 15750 50  0001 C CNN
+	1    15250 15750
+	1    0    0    -1
+$EndComp
+Wire Wire Line
+	15250 15750 15250 15700
+Wire Wire Line
+	15250 15700 15300 15700
+$Comp
+L Device:R R35
+U 1 1 62637E35
+P 15050 15600
+F 0 "R35" V 14843 15600 50  0000 C CNN
+F 1 "33R" V 14934 15600 50  0000 C CNN
+F 2 "Resistor_SMD:R_0603_1608Metric" V 14980 15600 50  0001 C CNN
+F 3 "~" H 15050 15600 50  0001 C CNN
+F 4 "C23140" H 15050 15600 50  0001 C CNN "LCSC"
+	1    15050 15600
+	0    1    1    0
+$EndComp
+Wire Wire Line
+	15300 15600 15200 15600
+Wire Wire Line
+	14900 15600 14850 15600
+Wire Wire Line
+	14850 15600 14850 14700
+Wire Wire Line
+	14850 14700 15200 14700
 $EndSCHEMATC
