File: hardware/rfboard/rfboard.kicad_sch (KiCad schematic)
At the start: 62 parts, among them J1 10118194-0001LF, J2 Conn_01x04, J3 2337019-1, J4 Conn_01x02, P2 CONN_01X03, SW1 SW_Push, SW2 SW_Push, SW3 SW_Push, U1 STM32G070KBTx, U2 RFM69HCW, U3 CH340X, U4 XL-0807RGBC-WS2812B, U5 XC6206P332MR-G, U6 HX 1210-C06

Commit message: Update rfboard KiCAD files to v9
Change-Id: I8b2d5b28951bb3e4204d908f966a681c3aa91492
Changed lines of the file:
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@@
 (kicad_sch
-	(version 20231120)
+	(version 20250114)
 	(generator "eeschema")
-	(generator_version "8.0")
+	(generator_version "9.0")
 	(paper "A3")
+	(text "5V -> 3.3V LDO"
+		(exclude_from_sim no)
+		(at 319.532 76.708 0)
+		(effects
+			(font
+				(size 1.27 1.27)
+			)
+		)
+	)
+	(text "USB connector\n(Power/programming)"
+		(exclude_from_sim no)
+		(at 255.778 62.738 0)
+		(effects
+			(font
+				(size 1.524 1.524)
+			)
+			(justify left bottom)
+		)
+	)
+	(text "rfboard"
+		(exclude_from_sim no)
+		(at 187.96 229.87 0)
+		(effects
+			(font
+				(size 1.524 1.524)
+			)
+			(justify left bottom)
+		)
+	)
+	(text "TIM14_CH1"
+		(exclude_from_sim no)
+		(at 45.466 61.468 0)
+		(effects
+			(font
+				(size 1.27 1.27)
+			)
+		)
+	)
+	(text "Offboard LED"
+		(exclude_from_sim no)
+		(at 36.322 199.644 0)
+		(effects
+			(font
+				(size 1.524 1.524)
+			)
+			(justify left bottom)
+		)
+	)
+	(text "SWD header"
+		(exclude_from_sim no)
+		(at 97.282 214.122 0)
+		(effects
+			(font
+				(size 1.27 1.27)
+			)
+		)
+	)
+	(text "SPI2_MOSI"
+		(exclude_from_sim no)
+		(at 127.508 53.848 0)
+		(effects
+			(font
+				(size 1.27 1.27)
+			)
+		)
+	)
+	(text "USB to serial"
+		(exclude_from_sim no)
+		(at 353.822 70.104 0)
+		(effects
+			(font
+				(size 1.27 1.27)
+			)
+		)
+	)
+	(text "\"One-click USB download\nof MCU\" configuration"
+		(exclude_from_sim no)
+		(at 390.144 20.066 0)
+		(effects
+			(font
+				(size 1.27 1.27)
+			)
+		)
+	)
+	(text "SPI1"
+		(exclude_from_sim no)
+		(at 47.498 69.342 0)
+		(effects
+			(font
+				(size 1.27 1.27)
+			)
+		)
+	)
+	(text "ADC_IN0"
+		(exclude_from_sim no)
+		(at 127.254 43.688 0)
+		(effects
+			(font
+				(size 1.27 1.27)
+			)
+		)
+	)
+	(text "TIM1_CH1"
+		(exclude_from_sim no)
+		(at 127.254 63.754 0)
+		(effects
+			(font
+				(size 1.27 1.27)
+			)
+		)
+	)
+	(text "BOOT0 == SWCLK"
+		(exclude_from_sim no)
+		(at 100.076 202.692 0)
+		(effects
+			(font
+				(size 1.27 1.27)
+			)
+		)
+	)
+	(text "Onboard LED"
+		(exclude_from_sim no)
+		(at 76.962 150.114 0)
+		(effects
+			(font
+				(size 1.27 1.27)
+			)
+		)
+	)
 	(junction
 		(at 45.72 52.07)
@@
 		)
 	)
-	(text "5V -> 3.3V LDO"
-		(exclude_from_sim no)
-		(at 319.532 76.708 0)
-		(effects
-			(font
-				(size 1.27 1.27)
-			)
-		)
-	)
-	(text "USB connector\n(Power/programming)"
-		(exclude_from_sim no)
-		(at 255.778 62.738 0)
-		(effects
-			(font
-				(size 1.524 1.524)
-			)
-			(justify left bottom)
-		)
-	)
-	(text "rfboard"
-		(exclude_from_sim no)
-		(at 187.96 229.87 0)
-		(effects
-			(font
-				(size 1.524 1.524)
-			)
-			(justify left bottom)
-		)
-	)
-	(text "TIM14_CH1"
-		(exclude_from_sim no)
-		(at 45.466 61.468 0)
-		(effects
-			(font
-				(size 1.27 1.27)
-			)
-		)
-	)
-	(text "Offboard LED"
-		(exclude_from_sim no)
-		(at 36.322 199.644 0)
-		(effects
-			(font
-				(size 1.524 1.524)
-			)
-			(justify left bottom)
-		)
-	)
-	(text "SWD header"
-		(exclude_from_sim no)
-		(at 97.282 214.122 0)
-		(effects
-			(font
-				(size 1.27 1.27)
-			)
-		)
-	)
-	(text "SPI2_MOSI"
-		(exclude_from_sim no)
-		(at 127.508 53.848 0)
-		(effects
-			(font
-				(size 1.27 1.27)
-			)
-		)
-	)
-	(text "USB to serial"
-		(exclude_from_sim no)
-		(at 353.822 70.104 0)
-		(effects
-			(font
-				(size 1.27 1.27)
-			)
-		)
-	)
-	(text "\"One-click USB download\nof MCU\" configuration"
-		(exclude_from_sim no)
-		(at 390.144 20.066 0)
-		(effects
-			(font
-				(size 1.27 1.27)
-			)
-		)
-	)
-	(text "SPI1"
-		(exclude_from_sim no)
-		(at 47.498 69.342 0)
-		(effects
-			(font
-				(size 1.27 1.27)
-			)
-		)
-	)
-	(text "ADC_IN0"
-		(exclude_from_sim no)
-		(at 127.254 43.688 0)
-		(effects
-			(font
-				(size 1.27 1.27)
-			)
-		)
-	)
-	(text "TIM1_CH1"
-		(exclude_from_sim no)
-		(at 127.254 63.754 0)
-		(effects
-			(font
-				(size 1.27 1.27)
-			)
-		)
-	)
-	(text "BOOT0 == SWCLK"
-		(exclude_from_sim no)
-		(at 100.076 202.692 0)
-		(effects
-			(font
-				(size 1.27 1.27)
-			)
-		)
-	)
-	(text "Onboard LED"
-		(exclude_from_sim no)
-		(at 76.962 150.114 0)
-		(effects
-			(font
-				(size 1.27 1.27)
-			)
-		)
-	)
 	(label "5V_DIVIDED"
 		(at 101.6 44.45 0)
@@
 		)
 		(instances
-			(project ""
+			(project "rfboard"
 				(path "/f88eb6ed-4fca-4205-8bd3-dd839e016fb0"
 					(reference "P2")
@@
 		)
 		(instances
-			(project ""
+			(project "rfboard"
 				(path "/f88eb6ed-4fca-4205-8bd3-dd839e016fb0"
 					(reference "#PWR01")
@@
 		)
 		(instances
-			(project ""
+			(project "rfboard"
 				(path "/f88eb6ed-4fca-4205-8bd3-dd839e016fb0"
 					(reference "#PWR02")
@@
 		)
 		(instances
-			(project ""
+			(project "rfboard"
 				(path "/f88eb6ed-4fca-4205-8bd3-dd839e016fb0"
 					(reference "#PWR04")
@@
 		)
 		(instances
-			(project ""
+			(project "rfboard"
 				(path "/f88eb6ed-4fca-4205-8bd3-dd839e016fb0"
 					(reference "#PWR05")
@@
 		)
 		(instances
-			(project ""
+			(project "rfboard"
 				(path "/f88eb6ed-4fca-4205-8bd3-dd839e016fb0"
 					(reference "#PWR07")
@@
 		)
 		(instances
-			(project ""
+			(project "rfboard"
 				(path "/f88eb6ed-4fca-4205-8bd3-dd839e016fb0"
 					(reference "#PWR013")
@@
 		)
 		(instances
-			(project ""
+			(project "rfboard"
 				(path "/f88eb6ed-4fca-4205-8bd3-dd839e016fb0"
 					(reference "J1")
@@
 		)
 		(instances
-			(project ""
+			(project "rfboard"
 				(path "/f88eb6ed-4fca-4205-8bd3-dd839e016fb0"
 					(reference "#PWR017")
@@
 		)
 		(instances
-			(project ""
+			(project "rfboard"
 				(path "/f88eb6ed-4fca-4205-8bd3-dd839e016fb0"
 					(reference "R2")
@@
 		)
 		(instances
-			(project ""
+			(project "rfboard"
 				(path "/f88eb6ed-4fca-4205-8bd3-dd839e016fb0"
 					(reference "#PWR032")
@@
 		)
 		(instances
-			(project ""
+			(project "rfboard"
 				(path "/f88eb6ed-4fca-4205-8bd3-dd839e016fb0"
 					(reference "H3")
@@
 		)
 		(instances
-			(project ""
+			(project "rfboard"
 				(path "/f88eb6ed-4fca-4205-8bd3-dd839e016fb0"
 					(reference "C7")
@@
 		)
 		(instances
-			(project ""
+			(project "rfboard"
 				(path "/f88eb6ed-4fca-4205-8bd3-dd839e016fb0"
 					(reference "L1")
@@
 		)
 		(instances
-			(project ""
+			(project "rfboard"
 				(path "/f88eb6ed-4fca-4205-8bd3-dd839e016fb0"
 					(reference "#PWR019")
@@
 		)
 		(instances
-			(project ""
+			(project "rfboard"
 				(path "/f88eb6ed-4fca-4205-8bd3-dd839e016fb0"
 					(reference "U4")
@@
 		)
 		(instances
-			(project ""
+			(project "rfboard"
 				(path "/f88eb6ed-4fca-4205-8bd3-dd839e016fb0"
 					(reference "U1")
@@
 		)
 		(instances
-			(project ""
+			(project "rfboard"
 				(path "/f88eb6ed-4fca-4205-8bd3-dd839e016fb0"
 					(reference "U6")
@@
 		)
 		(instances
-			(project ""
+			(project "rfboard"
 				(path "/f88eb6ed-4fca-4205-8bd3-dd839e016fb0"
 					(reference "U5")
@@
 		)
 		(instances
-			(project ""
+			(project "rfboard"
 				(path "/f88eb6ed-4fca-4205-8bd3-dd839e016fb0"
 					(reference "FB1")
@@
 		)
 		(instances
-			(project ""
+			(project "rfboard"
 				(path "/f88eb6ed-4fca-4205-8bd3-dd839e016fb0"
 					(reference "U3")
@@
 		)
 		(instances
-			(project ""
+			(project "rfboard"
 				(path "/f88eb6ed-4fca-4205-8bd3-dd839e016fb0"
 					(reference "J4")
@@
 		)
 		(instances
-			(project ""
+			(project "rfboard"
 				(path "/f88eb6ed-4fca-4205-8bd3-dd839e016fb0"
 					(reference "U2")
@@
 		)
 		(instances
-			(project ""
+			(project "rfboard"
 				(path "/f88eb6ed-4fca-4205-8bd3-dd839e016fb0"
 					(reference "#FLG1")
@@
 		)
 		(instances
-			(project ""
+			(project "rfboard"
 				(path "/f88eb6ed-4fca-4205-8bd3-dd839e016fb0"
 					(reference "J2")
@@
 		)
 	)
+	(embedded_fonts no)
 )
