File: hardware/rfboard/rfboard.kicad_sch (KiCad schematic)
At the start: 62 parts, among them J1 10118194-0001LF, J2 Conn_01x04, J3 2337019-1, J4 Conn_01x02, P2 CONN_01X03, SW1 SW_Push, SW2 SW_Push, SW3 SW_Push, U1 STM32G070KBTx, U2 RFM69HCW, U3 CH340X, U4 XL-0807RGBC-WS2812B, U5 XC6206P332MR-G, U6 HX 1210-C06

Commit message: Update the rfboard hardware designs for v2.1:
- Fix USB-USART connections to use the correct MCU pins
- Add thermal relief for the u.FL connector
- Switch to USB-C
- Switch to an LDO voltage regulator with a high PSRR
- Remove inner copper layers from antenna vias
- Increase antenna via copper to 1mm diameter
- Add a the 3rd pi filter footprint
- Add a 220uF electrolytic cap on the 5V rail
- Improve the decoupling story overall
- Remove the ferrite on the radio power supply

Change-Id: Iff05fab2d52248b6d165e85d5234a398977c2398
Parts:
- removed FB1: FerriteBead, Inductor_SMD:L_0603_1608Metric_Pad1.05x0.95mm_HandSolder, symbol Device:FerriteBead
- removed J2: Conn_01x04, Homebrew:PinHeader_1x04_P2.54mm_Vertical_NoPlastic, symbol Connector_Generic:Conn_01x04
- removed JP1: SolderJumper_2_Open, Jumper:SolderJumper-2_P1.3mm_Open_TrianglePad1.0x1.5mm, symbol Jumper:SolderJumper_2_Open
- removed U5: XC6206P332MR-G, Package_TO_SOT_SMD:SOT-23-3, symbol Regulator_Linear:XC6206PxxxMR
- added C27: 220uF, Capacitor_SMD:CP_Elec_6.3x5.8, symbol PCM_SparkFun-Capacitor:C_Polarized
- added C28, C29: 100nF, Capacitor_SMD:C_0402_1005Metric, symbol Device:C
- added L2: 0, Inductor_SMD:L_0402_1005Metric_Pad0.77x0.64mm_HandSolder, symbol Device:L
- added R12, R14: 5k1, Resistor_SMD:R_0402_1005Metric, symbol Device:R
- added R13, R15: 10k, Resistor_SMD:R_0402_1005Metric, symbol rfboard-rescue:R
- added U5: AP2112K-3.3, Package_TO_SOT_SMD:SOT-23-5, symbol Regulator_Linear:AP2112K-3.3
- C10, C15, C19: LCSC C96123 -> C426659
- C26: value 10uF -> 47uF; footprint Capacitor_SMD:C_0603_1608Metric -> Capacitor_SMD:C_1206_3216Metric; LCSC C96446 -> C426659
- C7: value 1pF -> 0R; LCSC C72134 -> C17168
- J1: footprint Homebrew:FRAMATOME_10118194-0001LF_fixed_bridges -> Homebrew:HRO_TYPE-C-31-M-12; symbol 10118194-0001LF:10118194-0001LF -> Homebrew:TYPE-C-31-M-12; LCSC C132563 -> C165948; MANUFACTURER (none) -> HRO Electronics; MAXIMUM_PACKAGE_HEIGHT (none) -> 3.31mm; PARTREV (none) -> A; STANDARD (none) -> Manufacturer Recommendations
- L1: value 10nH -> 0; LCSC C382409 -> (none); now not fitted
- U1: symbol MCU_ST_STM32G0:STM32G070KBTx -> Homebrew:STM32G070KBTx
Connections:
- net +3V3: now also C20.1, C26.2, C5.1, U2.13 (3.3V), U5.5 (VOUT); no longer C26.1
- net +5V: now also J1.A4B9 (VBUS), J1.B4A9 (VBUS), P2.3 (P3), C27.1, U5.1 (VIN), U5.3 (EN); no longer J1.1 (VDD), P2.1 (P1)
- net ANTENNA_UFL: now also C7.2, U2.9 (ANT), L2.1
- net GND: now also C26.1, J1.A1B12 (GND), J1.B1A12 (GND), J1.S1 (SHIELD), J1.S2 (SHIELD), J1.S3 (SHIELD), J1.S4 (SHIELD), P2.1 (P1), C27.2, C28.2, C29.2, L2.2, R12.2, R14.2, U5.2 (GND); no longer C26.2, J1.5 (GND), P2.3 (P3)
- net USART_RX: now also U1.21 (PA10); no longer U1.23 (PA10/PA12)
- net USART_TX: now also U1.19 (PA9); no longer U1.22 (PA9/PA11)
- net USB_DN: now also D3.1 (IO1), J1.A7 (DN1), J1.B7 (DN2); no longer D3.3 (IO2), J1.2 (D)
- net USB_DP: now also D3.3 (IO2), J1.A6 (DP1), J1.B6 (DP2); no longer D3.1 (IO1), J1.3 (D+)
- net CC2: now reaches U1.17 (PB2)
- net CC2: now also C29.1, R15.1
- net CC1: now reaches U1.8 (PA1)
- net CC1: now also C28.1, R13.2
- net CC2_RAW: now reaches D3.4 (IO3)
- net CC2_RAW: now also J1.B5 (CC2), R14.1, R15.2
- net CC1_RAW: now reaches D3.6 (IO4)
- net CC1_RAW: now also J1.A5 (CC1), R12.1, R13.1
- net SWDIO: no longer names the net of U1.24 (PA13)
Other:
- note removed: "BOOT0 == SWCLK"
- note removed: "SWD header"
- moved on the sheet: C10, C11, C12, C13, C14, C15, C16, C17, C18, C19, C20, C21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
